File: WiFiSTMBoard/WiFiSTMBoard.kicad_pcb (KiCad board)
At the start: 2 copper layers, 76 parts, among them J1 Conn_01x03_Male, J10 Conn_01x11_Male, J11 Conn_01x04_Male, J12 Conn_01x04_Male, J13 Conn_01x04_Male, J14 Conn_01x04_Male, J15 USB_B_Micro, J2 Conn_01x02_Male, J3 Conn_01x03_Male, J4 Conn_01x03_Male, J5 Conn_01x03_Male, J6 Conn_01x03_Male, J7 SWD, J9 Conn_01x06_Male, Q1 AO3401A, SW1 SW_Push_Dual_x2, SW2 PB12, SW3 PB14, SW4 PB13, SW5 PB15, U1 STM32F303RETx, U2 AMS1117-3.3, U3 USBLC6-2SC6, Y1 16MHz

Commit message: .
Parts:
- removed C8: 100n, Capacitor_SMD:C_0603_1608Metric
- removed J11, J13: Conn_01x04_Male, Connector_Molex:Molex_KK-396_A-41791-0004_1x04_P3.96mm_Vertical
- removed J6: Conn_01x03_Male, Connector_Molex:Molex_KK-396_A-41791-0003_1x03_P3.96mm_Vertical
- removed J9: Conn_01x06_Male, Connector_PinHeader_2.54mm:PinHeader_1x06_P2.54mm_Vertical
- removed TP2: TestPoint, TestPoint:TestPoint_Pad_D2.0mm
- removed TP7: TX4_TP, TestPoint:TestPoint_Pad_D2.0mm
- removed TP8: RX4_TP, TestPoint:TestPoint_Pad_D2.0mm
- added G***: LOGO, logo:ES, F.Cu at (123.5, 125.0)
- J12, J14: footprint Connector_Molex:Molex_KK-396_A-41791-0004_1x04_P3.96mm_Vertical -> Connector_PinHeader_2.54mm:PinHeader_1x04_P2.54mm_Horizontal
- J3, J4, J5: footprint Connector_Molex:Molex_KK-396_A-41791-0003_1x03_P3.96mm_Vertical -> Connector_Molex:Molex_Micro-Latch_53253-0370_1x03_P2.00mm_Vertical
- U1: value STM32F303RETx -> STM32F302C8Tx; footprint Package_QFP:LQFP-64_10x10mm_P0.5mm -> Package_QFP:LQFP-48_7x7mm_P0.5mm
- moved J10 143.1 mm to (77.2, 111.0), turned to 180 degrees
- moved J4 132.0 mm to (106.6, 133.0)
- moved J7 120.5 mm to (95.5, 84.3), turned to 270 degrees
- moved PA3 104.6 mm to (139.7, 127.0), turned to 180 degrees
- moved J5 104.1 mm to (117.0, 133.0)
- moved H1 102.0 mm to (145.0, 135.0)
- moved PA5 99.0 mm to (139.7, 111.8), turned to 180 degrees
- moved RST 97.9 mm to (89.4, 122.0), turned to 180 degrees
- moved PA4 92.5 mm to (139.7, 119.4), turned to 180 degrees
- moved D2 90.3 mm to (120.1, 116.2), turned to 90 degrees
- moved J12 84.2 mm to (144.8, 88.9)
- moved D1 80.4 mm to (122.7, 116.2), turned to 90 degrees
- moved H3 76.6 mm to (77.5, 135.0)
- moved C9 76.1 mm to (83.0, 122.0), turned to 270 degrees
- moved SW5 73.0 mm to (139.7, 104.1), turned to 180 degrees
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- renumbered SW2 to PA3, SW4 to PA4, SW3 to PA5, R12 to PA6, SW1 to RST
Connections:
- net Net-(U1-Pad17) renamed PA7
- net Net-(U1-Pad25) renamed PB12
- net Net-(U1-Pad26) renamed PB13
- net PC9_GPIO renamed PB4_GPIO
- C14 pad 1: PB12_BTN -> PA3_BTN
- C15 pad 1: PB14_BTN -> PA5_BTN
- C16 pad 1: PB13_BTN -> PA4_BTN
- C17 pad 1: PB15_BTN -> PA6_BTN
- J10 pad 1: +3V3 -> PC13
- J10 pad 10: PA9_GPIO -> Net-(J10-Pad10)
- J10 pad 11: PA10_GPIO -> Net-(J10-Pad11)
- J10 pad 2: GND -> PC14
- J10 pad 3: PC6_GPIO -> PC15
- J10 pad 4: PC7_GPIO -> PB6_GPIO
- J10 pad 5: PC8_GPIO -> PB5_GPIO
- J10 pad 7: VCC -> +3V3
- J10 pad 9: PA8_GPIO -> GND
- J12 pad 3: USART3_TX -> USART3_RX
- J12 pad 4: USART3_RX -> USART3_TX
- J14 pad 3: SCL -> SDA
- J14 pad 4: SDA -> SCL
- J5 pad 2: ADC1_CH6 -> ADC1_CH3
- PA3 pad 1: PB12_BTN -> PA3_BTN
- PA4 pad 1: PB13_BTN -> PA4_BTN
- PA5 pad 1: PB14_BTN -> PA5_BTN
- PA6 pad 2: PB15_BTN -> PA6_BTN
- R1 pad 1: LED_2 -> LED_1
- R11 pad 2: PB13_BTN -> PA4_BTN
- R7 pad 2: PB12_BTN -> PA3_BTN
- R8 pad 2: PB14_BTN -> PA5_BTN
- SW5 pad 1: PB15_BTN -> PA6_BTN
- U1 pad 10: Net-(U1-Pad10) -> ADC1_CH1
- U1 pad 11: Net-(U1-Pad11) -> ADC1_CH2
- U1 pad 12: GND -> ADC1_CH3
- U1 pad 13: +3.3VA -> PA3_BTN
- U1 pad 14: ADC1_CH1 -> PA4_BTN
- U1 pad 15: ADC1_CH2 -> PA5_BTN
- U1 pad 16: Net-(U1-Pad16) -> PA6_BTN
- U1 pad 18: GND -> LED_2
- U1 pad 19: +3V3 -> LED_1
- U1 pad 2: Net-(U1-Pad2) -> PC13
- U1 pad 20: PA4_GPIO -> PB2_GPIO
- U1 pad 21: PA5_GPIO -> USART3_TX
- U1 pad 22: PA6_GPIO -> USART3_RX
- U1 pad 23: PA7_GPIO -> GND
- U1 pad 24: Net-(U1-Pad24) -> +3V3
- U1 pad 27: LED_1 -> PB14
- U1 pad 28: LED_2 -> PB15
- U1 pad 29: USART3_TX -> PA8
- U1 pad 3: Net-(U1-Pad3) -> PC14
- U1 pad 30: USART3_RX -> UART1_TX
- U1 pad 31: GND -> UART1_RX
- U1 pad 32: +3V3 -> USB_DM
- U1 pad 33: PB12_BTN -> USB_DP
- U1 pad 34: PB13_BTN -> SWDIO
- U1 pad 35: PB14_BTN -> GND
- U1 pad 36: PB15_BTN -> +3V3
- U1 pad 37: PC6_GPIO -> SWCLK
- U1 pad 38: PC7_GPIO -> Net-(U1-Pad38)
- U1 pad 39: PC8_GPIO -> SWO
- U1 pad 4: Net-(U1-Pad4) -> PC15
- U1 pad 41: PA8_GPIO -> PB5_GPIO
- U1 pad 42: PA9_GPIO -> PB6_GPIO
- U1 pad 43: PA10_GPIO -> PB7_GPIO
- U1 pad 44: USB_DM -> BOOT0
- U1 pad 45: USB_DP -> SCL
- U1 pad 46: SWDIO -> SDA
- U1 pad 8: ADC1_CH6 -> GND
- U1 pad 9: ADC1_CH7 -> +3.3VA
Routing:
- net NRST: track 0.00 -> 97.4 mm, vias 0 -> 7
- net GND: track 0.00 -> 62.7 mm, vias 0 -> 38
- net PA3_BTN: track 0.00 -> 50.0 mm, vias 0 -> 2
- net PA4_BTN: track 0.00 -> 44.5 mm, vias 0 -> 2
- net +3V3: track 0.00 -> 43.5 mm, vias 0 -> 16
- net PA5_BTN: track 0.00 -> 41.5 mm, vias 0 -> 2
- net USART3_RX: track 0.00 -> 40.2 mm, vias 0 -> 1
- net USART3_TX: track 0.00 -> 39.8 mm, vias 0 -> 1
- net PA6_BTN: track 0.00 -> 37.8 mm, vias 0 -> 2
- net PC14: track 0.00 -> 37.0 mm, vias 0 -> 1
- net SCL: track 0.00 -> 37.0 mm
- net PB6_GPIO: track 0.00 -> 36.0 mm
- net SDA: track 0.00 -> 35.8 mm
- net PB4_GPIO: track 0.00 -> 35.3 mm
- net PC15: track 0.00 -> 34.9 mm, vias 0 -> 1
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- added copper zone on In2.Cu, net +3V3
- added copper zone on In1.Cu, net GND
Other:
- board outline added: 76.2 x 65.6 mm
- copper layers 2 -> 4
- board text added: "+"
- board text added: "-"
- board text added: "3.3"
- board text added: "3.3V"
- board text added: "3.3v"
- board text added: "ADC CH3"
- board text added: "ADC_CH1"
- board text added: "ADC_CH2"
- board text added: "BOOT0"
- board text added: "GND"
- board text added: "I2C1"
- board text added: "NC"
- board text added: "NRST"
- board text added: "PB4"
- board text added: "PB5"
- board text added: "PB6"
- board text added: "PC13"
- board text added: "PC14"
- board text added: "PC15"
- board text added: "POWER"
- board text added: "RX"
- board text added: "SCL"
- board text added: "SDA"
- board text added: "SWCLK"
- board text added: "SWDIO"
- board text added: "SWO"
- board text added: "TX"
- board text added: "UART3"
